File: Proto.sch (EAGLE design)
At the start: 1 part

Commit message: Adding additional circuits to schematic
Parts:
- added J1, J2: (no value), SparkFun-Connectors:CONN_04LOCK
- added J3: (no value), SparkFun-Connectors:CONN_03LOCK
- added J4, J5: (no value), SparkFun-Connectors:CONN_02LOCK
- added J6: (no value), SparkFun-Connectors:CONN_01
- added R1, R2, R3, R4: 1k, SparkFun-Resistors:1KOHM-HORIZ-1/4W-5%
- added R5: 600, SparkFun-Resistors:1KOHM-HORIZ-1/4W-5%
- added U$2, U$3: 2N3904, Carroll's Parts:2N3904
Connections:
- removed net 5V: U$1.DIR, U$1.VCC
- removed net GND: U$1.GND, U$1.OE
- new net K66F_3V: J3.2
- new net K66F_5V: J3.3, R2.2, R4.1, U$1.DIR, U$1.VCC, U$2.C
- new net K66F_GND: J3.1, U$1.GND, U$1.OE, U$2.E, U$3.E
- new net K66F_UART_RX: J5.2, R2.1, U$3.C
- new net K66F_UART_TX: J5.1, R3.2
- new net N$2: R4.2, U$3.B
- new net N$4: R1.2, U$2.B
- new net TK1_GND: J6.1, R5.1
- new net TK1_UART_RX: J4.2, R3.1, R5.2
- new net TK1_UART_TX: J4.1, R1.1
- net MOTOR_AA_3.3V: now also J1.1
- net MOTOR_AA_5V: now also J2.1
- net MOTOR_AB_3.3V: now also J1.2
- net MOTOR_AB_5V: now also J2.2
- net MOTOR_BA_3.3V: now also J1.3
- net MOTOR_BA_5V: now also J2.3
- net MOTOR_BB_3.3V: now also J1.4
- net MOTOR_BB_5V: now also J2.4
